Commit message: first commit

File: src/polebot_description/urdf/polebot.urdf.xacro (robot description, xacro)
@@ -160,5 +160,5 @@
   <!-- =================== SENSORS ============================ -->
   <!-- LiDAR frame -->
-  <link name="lidar_link">
+  <link name="laser">
     <visual>
       <geometry>
@@ -179,5 +179,5 @@
   <joint name="lidar_joint" type="fixed">
     <parent link="base_link"/>
-    <child  link="lidar_link"/>
+    <child  link="laser"/>
     <origin xyz="${base_length/4} 0 ${base_height/2 + 0.025}" rpy="0 0 0"/>
   </joint>

Commit message: feat: integrasi 3d model (meshes) dari branch diffdrive ke xacro main

File: src/polebot_description/urdf/polebot.urdf.xacro (robot description, xacro)
@@ -2,25 +2,34 @@
 <robot xmlns:xacro="http://www.ros.org/wiki/xacro" name="polebot">
   <!-- ======================================================== -->
-  <!--  POLEBOT — AMR Differential Drive Robot                  -->
+  <!--  POLEBOT � AMR Differential Drive Robot                  -->
   <!--  Politeknik Manufaktur Bandung                           -->
   <!-- ======================================================== -->
-  <!-- Include sub-components -->
   <xacro:include filename="$(find polebot_description)/urdf/materials.xacro"/>
-  <xacro:include filename="$(find polebot_description)/urdf/polebot_base.xacro"/>
-  <xacro:include filename="$(find polebot_description)/urdf/polebot_wheels.xacro"/>
-  <xacro:include filename="$(find polebot_description)/urdf/polebot_sensors.xacro"/>
   <!-- =================== ROBOT PARAMETERS =================== -->
-  <!-- Base dimensions -->
-  <xacro:property name="base_length"   value="0.45"/>   <!-- meters -->
-  <xacro:property name="base_width"    value="0.35"/>
-  <xacro:property name="base_height"   value="0.15"/>
-  <xacro:property name="base_mass"     value="8.0"/>    <!-- kg -->
+  <!-- Base dimensions (from CAD) -->
+  <xacro:property name="base_length"   value="1.172"/>
+  <xacro:property name="base_width"    value="0.670"/>
+  <xacro:property name="base_height"   value="0.563"/>
+  <xacro:property name="base_mass"     value="84.837"/>
   <!-- Wheel parameters -->
-  <xacro:property name="wheel_radius"  value="0.065"/>
-  <xacro:property name="wheel_width"   value="0.04"/>
-  <xacro:property name="wheel_mass"    value="0.5"/>
-  <xacro:property name="wheel_separation" value="0.35"/>
+  <xacro:property name="wheel_radius"  value="0.079"/>
+  <xacro:property name="wheel_width"   value="0.055"/>
+  <xacro:property name="wheel_mass"    value="3.610"/>
+  <xacro:property name="wheel_separation" value="0.600"/>
+  <xacro:property name="wheel_zoff"    value="0.231"/>
   <!-- Caster parameters -->
-  <xacro:property name="caster_radius" value="0.02"/>
+  <xacro:property name="caster_radius" value="0.0625"/>
+  <xacro:property name="caster_width"  value="0.0520"/>
+  <xacro:property name="caster_mass"   value="1.355"/>
+  <xacro:property name="caster_xoff"   value="0.300"/>
+  <xacro:property name="caster_yoff"   value="0.0289"/>
+  <xacro:property name="caster_zoff"   value="0.245"/>
+  <!-- Sensor parameters -->
+  <xacro:property name="lidar_xoff"    value="0.496"/>
+  <xacro:property name="lidar_zoff"    value="0.040"/>
+  <xacro:property name="camera_xoff"   value="0.560"/>
+  <xacro:property name="camera_zoff"   value="-0.023"/>
+  <xacro:property name="monitor_xoff"  value="0.204"/>
+  <xacro:property name="monitor_zoff"  value="0.730"/>
   <!-- =================== BASE FOOTPRINT ====================== -->
   <link name="base_footprint"/>
@@ -28,17 +37,19 @@
     <parent link="base_footprint"/>
     <child  link="base_link"/>
-    <origin xyz="0 0 ${wheel_radius}" rpy="0 0 0"/>
+    <origin xyz="0 0 ${wheel_radius + wheel_zoff}" rpy="0 0 0"/>
   </joint>
   <!-- =================== BASE LINK ========================== -->
   <link name="base_link">
     <visual>
-      <geometry>
-        <box size="${base_length} ${base_width} ${base_height}"/>
+      <origin xyz="0 0 0" rpy="0 0 0"/>
+      <geometry>
+        <mesh filename="package://polebot_description/meshes/polebot_amr.stl" scale="0.001 0.001 0.001"/>
       </geometry>
       <material name="dark_grey"/>
     </visual>
     <collision>
-      <geometry>
-        <box size="${base_length} ${base_width} ${base_height}"/>
+      <origin xyz="0 0 0" rpy="0 0 0"/>
+      <geometry>
+        <box size="${base_length} ${base_width} ${base_height/2}"/>
       </geometry>
     </collision>
@@ -53,125 +64,113 @@
     </inertial>
   </link>
-  <!-- =================== WHEELS ============================= -->
-  <!-- Left drive wheel -->
-  <link name="left_wheel_link">
-    <visual>
-      <geometry>
-        <cylinder radius="${wheel_radius}" length="${wheel_width}"/>
-      </geometry>
-      <material name="black"/>
-    </visual>
-    <collision>
-      <geometry>
-        <cylinder radius="${wheel_radius}" length="${wheel_width}"/>
-      </geometry>
-    </collision>
-    <inertial>
-      <mass value="${wheel_mass}"/>
-      <inertia
-        ixx="${(1/12)*wheel_mass*(3*wheel_radius**2 + wheel_width**2)}"
-        ixy="0" ixz="0"
-        iyy="${(1/2)*wheel_mass*wheel_radius**2}"
-        iyz="0"
-        izz="${(1/12)*wheel_mass*(3*wheel_radius**2 + wheel_width**2)}"/>
-    </inertial>
-  </link>
-  <joint name="left_wheel_joint" type="continuous">
-    <parent link="base_link"/>
-    <child  link="left_wheel_link"/>
-    <origin xyz="0 ${wheel_separation/2} 0" rpy="${-pi/2} 0 0"/>
-    <axis xyz="0 0 1"/>
-  </joint>
-  <!-- Right drive wheel -->
-  <link name="right_wheel_link">
-    <visual>
-      <geometry>
-        <cylinder radius="${wheel_radius}" length="${wheel_width}"/>
-      </geometry>
-      <material name="black"/>
-    </visual>
-    <collision>
-      <geometry>
-        <cylinder radius="${wheel_radius}" length="${wheel_width}"/>
-      </geometry>
-    </collision>
-    <inertial>
-      <mass value="${wheel_mass}"/>
-      <inertia
-        ixx="${(1/12)*wheel_mass*(3*wheel_radius**2 + wheel_width**2)}"
-        ixy="0" ixz="0"
-        iyy="${(1/2)*wheel_mass*wheel_radius**2}"
-        iyz="0"
-        izz="${(1/12)*wheel_mass*(3*wheel_radius**2 + wheel_width**2)}"/>
-    </inertial>
-  </link>
-  <joint name="right_wheel_joint" type="continuous">
-    <parent link="base_link"/>
-    <child  link="right_wheel_link"/>
-    <origin xyz="0 ${-wheel_separation/2} 0" rpy="${-pi/2} 0 0"/>
-    <axis xyz="0 0 1"/>
-  </joint>
-  <!-- Front caster -->
-  <link name="front_caster_link">
-    <visual>
-      <geometry>
-        <sphere radius="${caster_radius}"/>
-      </geometry>
-      <material name="white"/>
-    </visual>
-    <collision>
-      <geometry>
-        <sphere radius="${caster_radius}"/>
-      </geometry>
-    </collision>
-    <inertial>
-      <mass value="0.1"/>
-      <inertia ixx="0.0001" ixy="0" ixz="0" iyy="0.0001" iyz="0" izz="0.0001"/>
-    </inertial>
-  </link>
-  <joint name="front_caster_joint" type="fixed">
-    <parent link="base_link"/>
-    <child  link="front_caster_link"/>
-    <origin xyz="${base_length/2 - caster_radius} 0 ${-base_height/2 + caster_radius - wheel_radius}" rpy="0 0 0"/>
-  </joint>
-  <!-- Rear caster -->
-  <link name="rear_caster_link">
-    <visual>
-      <geometry>
-        <sphere radius="${caster_radius}"/>
-      </geometry>
-      <material name="white"/>
-    </visual>
-    <collision>
-      <geometry>
-        <sphere radius="${caster_radius}"/>
-      </geometry>
-    </collision>
-    <inertial>
-      <mass value="0.1"/>
-      <inertia ixx="0.0001" ixy="0" ixz="0" iyy="0.0001" iyz="0" izz="0.0001"/>
-    </inertial>
-  </link>
-  <joint name="rear_caster_joint" type="fixed">
-    <parent link="base_link"/>
-    <child  link="rear_caster_link"/>
-    <origin xyz="${-(base_length/2 - caster_radius)} 0 ${-base_height/2 + caster_radius - wheel_radius}" rpy="0 0 0"/>
-  </joint>
+  <!-- =================== MONITOR ============================ -->
+  <link name="monitor_link">
+    <visual>
+      <origin xyz="0 0 0" rpy="0 0 0"/>
+      <geometry>
+        <mesh filename="package://polebot_description/meshes/monitor.stl" scale="0.001 0.001 0.001"/>
+      </geometry>
+      <material name="dark_grey"/>
+    </visual>
+    <collision>
+      <origin xyz="0 0 0" rpy="0 0 0"/>
+      <geometry>
+        <box size="0.1 0.1 0.9"/>
+      </geometry>
+    </collision>
+    <inertial>
+      <mass value="16.008"/>
+      <inertia ixx="0.1" ixy="0" ixz="0" iyy="0.1" iyz="0" izz="0.1"/>
+    </inertial>
+  </link>
+  <joint name="monitor_joint" type="fixed">
+    <parent link="base_link"/>
+    <child link="monitor_link"/>
+    <origin xyz="${monitor_xoff} 0 ${monitor_zoff}" rpy="0 0 0"/>
+  </joint>
+  <!-- =================== WHEELS MACRO ======================= -->
+  <xacro:macro name="drive_wheel" params="prefix y_reflect">
+    <link name="${prefix}_link">
+      <visual>
+        <origin xyz="0 0 0" rpy="0 0 ${(y_reflect-1)*pi/2}"/>
+        <geometry>
+          <mesh filename="package://polebot_description/meshes/wheel.stl" scale="0.001 0.001 0.001"/>
+        </geometry>
+        <material name="black"/>
+      </visual>
+      <collision>
+        <origin xyz="0 0 0" rpy="${pi/2} 0 0"/>
+        <geometry>
+          <cylinder radius="${wheel_radius}" length="${wheel_width}"/>
+        </geometry>
+      </collision>
+      <inertial>
+        <mass value="${wheel_mass}"/>
+        <inertia
+          ixx="${(1/12)*wheel_mass*(3*wheel_radius**2 + wheel_width**2)}"
+          ixy="0" ixz="0"
+          iyy="${(1/2)*wheel_mass*wheel_radius**2}"
+          iyz="0"
+          izz="${(1/12)*wheel_mass*(3*wheel_radius**2 + wheel_width**2)}"/>
+      </inertial>
+    </link>
+    <joint name="${prefix}_joint" type="continuous">
+      <parent link="base_link"/>
+      <child  link="${prefix}_link"/>
+      <origin xyz="0 ${y_reflect * wheel_separation/2} ${-wheel_zoff}" rpy="0 0 0"/>
+      <axis xyz="0 1 0"/>
+    </joint>
+  </xacro:macro>
+  <xacro:drive_wheel prefix="drivewhl_l" y_reflect="1"/>
+  <xacro:drive_wheel prefix="drivewhl_r" y_reflect="-1"/>
+  <!-- =================== CASTER MACRO ======================= -->
+  <xacro:macro name="caster_wheel" params="prefix x_reflect y_reflect">
+    <link name="${prefix}_link">
+      <visual>
+        <origin xyz="0 0 0" rpy="0 0 0"/>
+        <geometry>
+          <mesh filename="package://polebot_description/meshes/caster.stl" scale="0.001 0.001 0.001"/>
+        </geometry>
+        <material name="white"/>
+      </visual>
+      <collision>
+        <origin xyz="0 0 0" rpy="0 0 0"/>
+        <geometry>
+          <sphere radius="${caster_radius}"/>
+        </geometry>
+      </collision>
+      <inertial>
+        <mass value="${caster_mass}"/>
+        <inertia ixx="0.001" ixy="0" ixz="0" iyy="0.001" iyz="0" izz="0.001"/>
+      </inertial>
+    </link>
+    <joint name="${prefix}_joint" type="fixed">
+      <parent link="base_link"/>
+      <child  link="${prefix}_link"/>
+      <origin xyz="${x_reflect * caster_xoff} ${y_reflect * (base_width/2 + caster_yoff)} ${-caster_zoff}" rpy="0 0 0"/>
+    </joint>
+  </xacro:macro>
+  <xacro:caster_wheel prefix="casterwhl_fl" x_reflect="1" y_reflect="1"/>
+  <xacro:caster_wheel prefix="casterwhl_fr" x_reflect="1" y_reflect="-1"/>
+  <xacro:caster_wheel prefix="casterwhl_rl" x_reflect="-1" y_reflect="1"/>
+  <xacro:caster_wheel prefix="casterwhl_rr" x_reflect="-1" y_reflect="-1"/>
   <!-- =================== SENSORS ============================ -->
   <!-- LiDAR frame -->
-  <link name="laser">
-    <visual>
-      <geometry>
-        <cylinder radius="0.035" length="0.045"/>
+  <link name="lidar_link">
+    <visual>
+      <origin xyz="0 0 0" rpy="0 0 0"/>
+      <geometry>
+        <mesh filename="package://polebot_description/meshes/lidar.stl" scale="0.001 0.001 0.001"/>
       </geometry>
       <material name="blue"/>
     </visual>
     <collision>
-      <geometry>
-        <cylinder radius="0.035" length="0.045"/>
-      </geometry>
-    </collision>
-    <inertial>
-      <mass value="0.2"/>
+      <origin xyz="0 0 0" rpy="0 0 0"/>
+      <geometry>
+        <cylinder radius="0.0208" length="0.055"/>
+      </geometry>
+    </collision>
+    <inertial>
+      <mass value="0.125"/>
       <inertia ixx="0.0001" ixy="0" ixz="0" iyy="0.0001" iyz="0" izz="0.0001"/>
     </inertial>
@@ -179,6 +178,6 @@
   <joint name="lidar_joint" type="fixed">
     <parent link="base_link"/>
-    <child  link="laser"/>
-    <origin xyz="${base_length/4} 0 ${base_height/2 + 0.025}" rpy="0 0 0"/>
+    <child  link="lidar_link"/>
+    <origin xyz="${lidar_xoff} 0 ${lidar_zoff}" rpy="0 0 0"/>
   </joint>
   <!-- IMU frame -->
@@ -192,21 +191,23 @@
     <parent link="base_link"/>
     <child  link="imu_link"/>
-    <origin xyz="0 0 0" rpy="0 0 0"/>
+    <origin xyz="0.1 0 0.1" rpy="0 0 0"/>
   </joint>
   <!-- Camera frame -->
   <link name="camera_link">
     <visual>
-      <geometry>
-        <box size="0.025 0.09 0.025"/>
+      <origin xyz="0 0 0" rpy="0 0 0"/>
+      <geometry>
+        <mesh filename="package://polebot_description/meshes/camera.stl" scale="0.001 0.001 0.001"/>
       </geometry>
       <material name="dark_grey"/>
     </visual>
     <collision>
-      <geometry>
-        <box size="0.025 0.09 0.025"/>
-      </geometry>
-    </collision>
-    <inertial>
-      <mass value="0.1"/>
+      <origin xyz="0 0 0" rpy="0 0 0"/>
+      <geometry>
+        <box size="0.015 0.130 0.0222"/>
+      </geometry>
+    </collision>
+    <inertial>
+      <mass value="0.123"/>
       <inertia ixx="0.0001" ixy="0" ixz="0" iyy="0.0001" iyz="0" izz="0.0001"/>
     </inertial>
@@ -215,5 +216,5 @@
     <parent link="base_link"/>
     <child  link="camera_link"/>
-    <origin xyz="${base_length/2} 0 ${base_height/4}" rpy="0 0 0"/>
+    <origin xyz="${camera_xoff} 0 ${camera_zoff}" rpy="0 0 0"/>
   </joint>
   <link name="camera_optical_frame"/>

Commit message: fix: koreksi orientasi lidar (-90 deg) dan trust_odom di slam_toolbox

File: src/polebot_description/urdf/polebot.urdf.xacro (robot description, xacro)
@@ -179,5 +179,5 @@
     <parent link="base_link"/>
     <child  link="lidar_link"/>
-    <origin xyz="${lidar_xoff} 0 ${lidar_zoff}" rpy="0 0 0"/>
+    <origin xyz="${lidar_xoff} 0 ${lidar_zoff}" rpy="0 0 -${pi/2}"/>
   </joint>
   <!-- IMU frame -->

Commit message: feat: Add Nav2 Zone Editor UI and Backend integration for keepout and speed zones

File: src/polebot_description/urdf/polebot.urdf.xacro (robot description, xacro)
@@ -2,8 +2,9 @@
 <robot xmlns:xacro="http://www.ros.org/wiki/xacro" name="polebot">
   <!-- ======================================================== -->
-  <!--  POLEBOT � AMR Differential Drive Robot                  -->
+  <!--  POLEBOT - AMR Differential Drive Robot                  -->
   <!--  Politeknik Manufaktur Bandung                           -->
   <!-- ======================================================== -->
   <xacro:include filename="$(find polebot_description)/urdf/materials.xacro"/>
+  <xacro:include filename="$(find polebot_description)/urdf/polebot.gazebo.xacro"/>
   <!-- =================== ROBOT PARAMETERS =================== -->
   <!-- Base dimensions (from CAD) -->
@@ -157,5 +158,5 @@
   <!-- =================== SENSORS ============================ -->
   <!-- LiDAR frame -->
-  <link name="lidar_link">
+  <link name="laser">
     <visual>
       <origin xyz="0 0 0" rpy="0 0 0"/>
@@ -176,8 +177,8 @@
     </inertial>
   </link>
-  <joint name="lidar_joint" type="fixed">
-    <parent link="base_link"/>
-    <child  link="lidar_link"/>
-    <origin xyz="${lidar_xoff} 0 ${lidar_zoff}" rpy="0 0 -${pi/2}"/>
+  <joint name="laser_joint" type="fixed">
+    <parent link="base_link"/>
+    <child  link="laser"/>
+    <origin xyz="${lidar_xoff} 0 ${lidar_zoff}" rpy="0 0 ${-pi/2}"/>
   </joint>
   <!-- IMU frame -->
